Commit message: Description package done till now...

File: ros2_ws/src/robotic-arm_description/urdf/robotic-arm.xacro (robot description, xacro)
@@ -1,4 +1,8 @@
 <?xml version='1.0' encoding='utf-8'?>
-<robot name="robotic_arm">
+<robot name="robotic-arm" xmlns:xacro="http://www.ros.org/wiki/xacro">
+  <!-- Include materials -->
+  <xacro:include filename="$(find robotic-arm_description)/urdf/materials.xacro"/>
+  <!-- Include gazebo -->
+  <!-- <xacro:include filename="$(find robotic-arm_description)/urdf/gazebo.xacro"/> -->
     <link name="base_footprint"/>
     <link name="base_link">
@@ -11,11 +15,12 @@
             <origin xyz="0.0 0.0 0.0" rpy="0.0 0.0 0.0" />
             <geometry>
-                <mesh filename="file://($find robotic-arm_description)/meshes/base_link.stl" scale="0.001 0.001 0.001" />
-            </geometry>
+                <mesh filename="package://robotic-arm_description/meshes/base_link.stl" scale="0.001 0.001 0.001" />
+            </geometry>
+            <material name="Base_link"/>
         </visual>
         <collision name="base_link_collision">
             <origin xyz="0.0 0.0 0.0" rpy="0.0 0.0 0.0" />
             <geometry>
-                <mesh filename="file://($find robotic-arm_description)/meshes/base_link.stl" scale="0.001 0.001 0.001" />
+                <mesh filename="package://robotic-arm_description/meshes/base_link.stl" scale="0.001 0.001 0.001" />
             </geometry>
         </collision>
@@ -30,11 +35,12 @@
             <origin xyz="0.0 0.0 0.01" rpy="0.0 -0.0 0.0" />
             <geometry>
-                <mesh filename="file://($find robotic-arm_description)/meshes/base.stl" scale="0.001 0.001 0.001" />
-            </geometry>
+                <mesh filename="package://robotic-arm_description/meshes/base.stl" scale="0.001 0.001 0.001" />
+            </geometry>
+            <material name="Base"/>
         </visual>
         <collision name="base_collision">
             <origin xyz="0.0 0.0 0.01" rpy="0.0 -0.0 0.0" />
             <geometry>
-                <mesh filename="file://($find robotic-arm_description)/meshes/base.stl" scale="0.001 0.001 0.001" />
+                <mesh filename="package://robotic-arm_description/meshes/base.stl" scale="0.001 0.001 0.001" />
             </geometry>
         </collision>
@@ -49,11 +55,12 @@
             <origin xyz="0.021920310543421046 0.021920310543421053 -1.1102230246251566e-18" rpy="1.5707963267948966 2.7755575615628907e-17 -0.7853981633974483" />
             <geometry>
-                <mesh filename="file://($find robotic-arm_description)/meshes/arm_link.stl" scale="0.001 0.001 0.001" />
-            </geometry>
+                <mesh filename="package://robotic-arm_description/meshes/arm_link.stl" scale="0.001 0.001 0.001" />
+            </geometry>
+            <material name="arm"/>
         </visual>
         <collision name="arm_link_collision">
             <origin xyz="0.021920310543421046 0.021920310543421053 -1.1102230246251566e-18" rpy="1.5707963267948966 2.7755575615628907e-17 -0.7853981633974483" />
             <geometry>
-                <mesh filename="file://($find robotic-arm_description)/meshes/arm_link.stl" scale="0.001 0.001 0.001" />
+                <mesh filename="package://robotic-arm_description/meshes/arm_link.stl" scale="0.001 0.001 0.001" />
             </geometry>
         </collision>
@@ -68,11 +75,12 @@
             <origin xyz="-0.16581654376326369 0.16581654021678285 7.549516567451074e-17" rpy="1.570796326794897 -1.110223024625157e-16 0.7853981633974477" />
             <geometry>
-                <mesh filename="file://($find robotic-arm_description)/meshes/forearm_link.stl" scale="0.001 0.001 0.001" />
-            </geometry>
+                <mesh filename="package://robotic-arm_description/meshes/forearm_link.stl" scale="0.001 0.001 0.001" />
+            </geometry>
+            <material name="forearm"/>
         </visual>
         <collision name="forearm_link_collision">
             <origin xyz="-0.16581654376326369 0.16581654021678285 7.549516567451074e-17" rpy="1.570796326794897 -1.110223024625157e-16 0.7853981633974477" />
             <geometry>
-                <mesh filename="file://($find robotic-arm_description)/meshes/forearm_link.stl" scale="0.001 0.001 0.001" />
+                <mesh filename="package://robotic-arm_description/meshes/forearm_link.stl" scale="0.001 0.001 0.001" />
             </geometry>
         </collision>
@@ -87,11 +95,12 @@
             <origin xyz="-0.442500003834537 -2.2600423932317426e-09 4.440892098500637e-18" rpy="1.5707963267948968 -2.747661802696606e-16 1.5707963267948966" />
             <geometry>
-                <mesh filename="file://($find robotic-arm_description)/meshes/wrist_link.stl" scale="0.001 0.001 0.001" />
-            </geometry>
+                <mesh filename="package://robotic-arm_description/meshes/wrist_link.stl" scale="0.001 0.001 0.001" />
+            </geometry>
+            <material name="wrist"/>
         </visual>
         <collision name="wrist_link_collision">
             <origin xyz="-0.442500003834537 -2.2600423932317426e-09 4.440892098500637e-18" rpy="1.5707963267948968 -2.747661802696606e-16 1.5707963267948966" />
             <geometry>
-                <mesh filename="file://($find robotic-arm_description)/meshes/wrist_link.stl" scale="0.001 0.001 0.001" />
+                <mesh filename="package://robotic-arm_description/meshes/wrist_link.stl" scale="0.001 0.001 0.001" />
             </geometry>
         </collision>
@@ -106,11 +115,12 @@
             <origin xyz="-0.5014000038345371 4.440892098500626e-18 2.2600423932317426e-09" rpy="1.177569344012831e-16 1.5707963267948963 0" />
             <geometry>
-                <mesh filename="file://($find robotic-arm_description)/meshes/gripper_link.stl" scale="0.001 0.001 0.001" />
-            </geometry>
+                <mesh filename="package://robotic-arm_description/meshes/gripper_link.stl" scale="0.001 0.001 0.001" />
+            </geometry>
+            <material name="gripper"/>
         </visual>
         <collision name="gripper_link_collision">
             <origin xyz="-0.5014000038345371 4.440892098500626e-18 2.2600423932317426e-09" rpy="1.177569344012831e-16 1.5707963267948963 0" />
             <geometry>
-                <mesh filename="file://($find robotic-arm_description)/meshes/gripper_link.stl" scale="0.001 0.001 0.001" />
+                <mesh filename="package://robotic-arm_description/meshes/gripper_link.stl" scale="0.001 0.001 0.001" />
             </geometry>
         </collision>
@@ -125,11 +135,12 @@
             <origin xyz="-0.5024000038345371 -0.007499999999999995 0.010000002260042358" rpy="1.177569344012831e-16 1.5707963267948963 0" />
             <geometry>
-                <mesh filename="file://($find robotic-arm_description)/meshes/finger_l.stl" scale="0.001 0.001 0.001" />
-            </geometry>
+                <mesh filename="package://robotic-arm_description/meshes/finger_l.stl" scale="0.001 0.001 0.001" />
+            </geometry>
+            <material name="gripper"/>
         </visual>
         <collision name="finger_l_collision">
             <origin xyz="-0.5024000038345371 -0.007499999999999995 0.010000002260042358" rpy="1.177569344012831e-16 1.5707963267948963 0" />
             <geometry>
-                <mesh filename="file://($find robotic-arm_description)/meshes/finger_l.stl" scale="0.001 0.001 0.001" />
+                <mesh filename="package://robotic-arm_description/meshes/finger_l.stl" scale="0.001 0.001 0.001" />
             </geometry>
         </collision>
@@ -144,11 +155,12 @@
             <origin xyz="-0.5024000038345371 0.007500000000000005 -0.009999997739957607" rpy="1.177569344012831e-16 1.5707963267948963 0" />
             <geometry>
-                <mesh filename="file://($find robotic-arm_description)/meshes/finger_r.stl" scale="0.001 0.001 0.001" />
-            </geometry>
+                <mesh filename="package://robotic-arm_description/meshes/finger_r.stl" scale="0.001 0.001 0.001" />
+            </geometry>
+            <material name="gripper"/>
         </visual>
         <collision name="finger_r_collision">
             <origin xyz="-0.5024000038345371 0.007500000000000005 -0.009999997739957607" rpy="1.177569344012831e-16 1.5707963267948963 0" />
             <geometry>
-                <mesh filename="file://($find robotic-arm_description)/meshes/finger_r.stl" scale="0.001 0.001 0.001" />
+                <mesh filename="package://robotic-arm_description/meshes/finger_r.stl" scale="0.001 0.001 0.001" />
             </geometry>
         </collision>
@@ -160,5 +172,5 @@
         <axis xyz="0.0 0.0 1.0" />
     </joint>
-    <joint name="base_link_base_rotation" type="continuous">
+    <joint name="base_rotation" type="continuous">
         <origin xyz="0.0 0.0 -0.01" rpy="0.0 -0.0 0.0" />
         <parent link="base_link" />
@@ -166,5 +178,5 @@
         <axis xyz="0.0 0.0 1.0" />
     </joint>
-    <joint name="base_arm_rotation" type="continuous">
+    <joint name="arm_rotation" type="continuous">
         <origin xyz="0.0 0.0 0.040999999999999995" rpy="-1.5707963267948966 -0.0 0.0" />
         <parent link="base" />
@@ -172,5 +184,5 @@
         <axis xyz="0.0 0.0 1.0" />
     </joint>
-    <joint name="arm_link_forearm_rotation" type="continuous">
+    <joint name="forearm_rotation" type="continuous">
         <origin xyz="-0.14389623 -0.14389623 0.0" rpy="1.3866695599588117e-32 -2.5658541216885115e-48 0.0" />
         <parent link="arm_link" />
@@ -178,5 +190,5 @@
         <axis xyz="2.5658541216885078e-48 1.3866695599588098e-32 0.9999999999999987" />
     </joint>
-    <joint name="forearm_link_wrist_rotation" type="continuous">
+    <joint name="wrist_rotation" type="continuous">
         <origin xyz="0.14707821000000024 -0.14707820999999996 2.0394887674022966e-33" rpy="-1.38666955995881e-32 -2.4651903288156613e-32 -1.1344072614353854e-48" />
         <parent link="forearm_link" />
@@ -189,17 +201,17 @@
         <child link="gripper_link" />
     </joint>
-    <joint name="gripper_link_finger_l_joint" type="prismatic">
+    <joint name="finger_r_joint" type="prismatic">
         <origin xyz="0.0002499999999999947 0.0 0.01" rpy="0.0 -0.0 0.0" />
         <parent link="gripper_link" />
         <child link="finger_r" />
         <axis xyz="0.0 1.0 0.0" />
-        <limit lower="100" upper="100" effort="50" velocity="1"/>
-    </joint>
-    <joint name="gripper_link_finger_r_joint" type="prismatic">
+        <limit lower="0" upper="0" effort="50" velocity="1"/>
+    </joint>
+    <joint name="finger_l_joint" type="prismatic">
         <origin xyz="0.0002499999999999947 0.0 -0.009999999999999966" rpy="0.0 -0.0 0.0" />
         <parent link="gripper_link" />
         <child link="finger_l" />
         <axis xyz="-0.0 -1.0 -0.0" />
-        <limit lower="100" upper="100" effort="50" velocity="1"/>
+        <limit lower="0" upper="0" effort="50" velocity="1"/>
     </joint>
 </robot>
